Commit message: republish model

File: urdf/ros_robot.xacro (robot description, xacro)
@@ -6,7 +6,7 @@
 <link name="base_link">
   <inertial>
-    <origin xyz="0.007676097193994553 -3.022810042874328e-06 0.02223666734325978" rpy="0 0 0"/>
-    <mass value="0.8806285630036556"/>
-    <inertia ixx="0.000282" iyy="0.0008" izz="0.000719" ixy="0.0" iyz="0.0" ixz="5.6e-05"/>
+    <origin xyz="0.044354227312182234 0.08057379028516376 0.21043007492326804" rpy="0 0 0"/>
+    <mass value="880.6995319303643"/>
+    <inertia ixx="28.28545" iyy="80.038922" izz="71.915121" ixy="0.008323" iyz="0.00454" ixz="5.656101"/>
   </inertial>
   <visual>
@@ -26,10 +26,10 @@
 <link name="CenterThrusterR_1">
   <inertial>
-    <origin xyz="-3.359918489195812e-07 0.0020000000000000018 -7.551522476778594e-09" rpy="0 0 0"/>
-    <mass value="0.0024661502330678834"/>
-    <inertia ixx="0.0" iyy="0.0" izz="0.0" ixy="0.0" iyz="0.0" ixz="-0.0"/>
-  </inertial>
-  <visual>
-    <origin xyz="0.033569 -0.003 -0.011066" rpy="0 0 0"/>
+    <origin xyz="3.8493357595870137e-07 0.020000218269361866 -7.552568147273231e-08" rpy="0 0 0"/>
+    <mass value="2.4661502330679896"/>
+    <inertia ixx="0.00187" iyy="0.003083" izz="0.00187" ixy="-0.0" iyz="-0.0" ixz="-0.0"/>
+  </inertial>
+  <visual>
+    <origin xyz="0.368081 -0.110604 -0.09866" rpy="0 0 0"/>
     <geometry>
       <mesh filename="package://ros_robot_description/meshes/CenterThrusterR_1.stl" scale="0.001 0.001 0.001"/>
@@ -38,5 +38,5 @@
   </visual>
   <collision>
-    <origin xyz="0.033569 -0.003 -0.011066" rpy="0 0 0"/>
+    <origin xyz="0.368081 -0.110604 -0.09866" rpy="0 0 0"/>
     <geometry>
       <mesh filename="package://ros_robot_description/meshes/CenterThrusterR_1.stl" scale="0.001 0.001 0.001"/>
@@ -46,10 +46,10 @@
 <link name="CenterThrusterL_1">
   <inertial>
-    <origin xyz="-3.359918489195812e-07 -0.0019999999999999974 -7.551522476778594e-09" rpy="0 0 0"/>
-    <mass value="0.0024661502330678834"/>
-    <inertia ixx="0.0" iyy="0.0" izz="0.0" ixy="0.0" iyz="-0.0" ixz="-0.0"/>
-  </inertial>
-  <visual>
-    <origin xyz="0.033569 0.003 -0.011066" rpy="0 0 0"/>
+    <origin xyz="3.849335762362571e-07 -0.01999978173063812 -7.552568151436567e-08" rpy="0 0 0"/>
+    <mass value="2.4661502330679888"/>
+    <inertia ixx="0.00187" iyy="0.003083" izz="0.00187" ixy="0.0" iyz="-0.0" ixz="0.0"/>
+  </inertial>
+  <visual>
+    <origin xyz="0.368081 -0.050604 -0.09866" rpy="0 0 0"/>
     <geometry>
       <mesh filename="package://ros_robot_description/meshes/CenterThrusterL_1.stl" scale="0.001 0.001 0.001"/>
@@ -58,5 +58,5 @@
   </visual>
   <collision>
-    <origin xyz="0.033569 0.003 -0.011066" rpy="0 0 0"/>
+    <origin xyz="0.368081 -0.050604 -0.09866" rpy="0 0 0"/>
     <geometry>
       <mesh filename="package://ros_robot_description/meshes/CenterThrusterL_1.stl" scale="0.001 0.001 0.001"/>
@@ -66,10 +66,10 @@
 <link name="BackThrusterR_1">
   <inertial>
-    <origin xyz="0.0029999999999999957 3.469446951953614e-18 4.933727255239037e-07" rpy="0 0 0"/>
-    <mass value="0.005326884503426852"/>
-    <inertia ixx="0.0" iyy="0.0" izz="0.0" ixy="-0.0" iyz="0.0" ixz="0.0"/>
-  </inertial>
-  <visual>
-    <origin xyz="-0.051 -0.01 -0.007554" rpy="0 0 0"/>
+    <origin xyz="0.029999744852065302 2.182693619456888e-07 -6.627274470871747e-08" rpy="0 0 0"/>
+    <mass value="5.326884503426855"/>
+    <inertia ixx="0.009588" iyy="0.006392" izz="0.006392" ixy="0.0" iyz="0.0" ixz="0.0"/>
+  </inertial>
+  <visual>
+    <origin xyz="-0.477613 -0.180604 -0.063545" rpy="0 0 0"/>
     <geometry>
       <mesh filename="package://ros_robot_description/meshes/BackThrusterR_1.stl" scale="0.001 0.001 0.001"/>
@@ -78,5 +78,5 @@
   </visual>
   <collision>
-    <origin xyz="-0.051 -0.01 -0.007554" rpy="0 0 0"/>
+    <origin xyz="-0.477613 -0.180604 -0.063545" rpy="0 0 0"/>
     <geometry>
       <mesh filename="package://ros_robot_description/meshes/BackThrusterR_1.stl" scale="0.001 0.001 0.001"/>
@@ -86,10 +86,10 @@
 <link name="BackThrusterL_1">
   <inertial>
-    <origin xyz="0.0029999999999999957 6.938893903907228e-18 4.933727255239037e-07" rpy="0 0 0"/>
-    <mass value="0.005326884503426849"/>
-    <inertia ixx="0.0" iyy="0.0" izz="0.0" ixy="0.0" iyz="0.0" ixz="0.0"/>
-  </inertial>
-  <visual>
-    <origin xyz="-0.051 0.01 -0.007554" rpy="0 0 0"/>
+    <origin xyz="0.02999974485206519 2.1826936186936097e-07 -6.627274470871747e-08" rpy="0 0 0"/>
+    <mass value="5.3268845034268555"/>
+    <inertia ixx="0.009588" iyy="0.006392" izz="0.006392" ixy="-0.0" iyz="-0.0" ixz="0.0"/>
+  </inertial>
+  <visual>
+    <origin xyz="-0.477613 0.019396 -0.063545" rpy="0 0 0"/>
     <geometry>
       <mesh filename="package://ros_robot_description/meshes/BackThrusterL_1.stl" scale="0.001 0.001 0.001"/>
@@ -98,5 +98,5 @@
   </visual>
   <collision>
-    <origin xyz="-0.051 0.01 -0.007554" rpy="0 0 0"/>
+    <origin xyz="-0.477613 0.019396 -0.063545" rpy="0 0 0"/>
     <geometry>
       <mesh filename="package://ros_robot_description/meshes/BackThrusterL_1.stl" scale="0.001 0.001 0.001"/>
@@ -106,10 +106,10 @@
 <link name="JawL_1">
   <inertial>
-    <origin xyz="0.0031886327495435976 -0.0010363707756858593 -0.002669458127535926" rpy="0 0 0"/>
-    <mass value="0.00018598053770556956"/>
-    <inertia ixx="0.0" iyy="0.0" izz="0.0" ixy="0.0" iyz="-0.0" ixz="0.0"/>
-  </inertial>
-  <visual>
-    <origin xyz="-0.060082 -0.007875 -0.072623" rpy="0 0 0"/>
+    <origin xyz="0.03189007234749497 -0.010365489487497326 -0.026698581275366062" rpy="0 0 0"/>
+    <mass value="0.18598053770557255"/>
+    <inertia ixx="7e-05" iyy="0.000135" izz="9.2e-05" ixy="1.7e-05" iyz="-1.4e-05" ixz="6.3e-05"/>
+  </inertial>
+  <visual>
+    <origin xyz="-0.568429 -0.159356 -0.714234" rpy="0 0 0"/>
     <geometry>
       <mesh filename="package://ros_robot_description/meshes/JawL_1.stl" scale="0.001 0.001 0.001"/>
@@ -118,5 +118,5 @@
   </visual>
   <collision>
-    <origin xyz="-0.060082 -0.007875 -0.072623" rpy="0 0 0"/>
+    <origin xyz="-0.568429 -0.159356 -0.714234" rpy="0 0 0"/>
     <geometry>
       <mesh filename="package://ros_robot_description/meshes/JawL_1.stl" scale="0.001 0.001 0.001"/>
@@ -126,10 +126,10 @@
 <link name="JawR_1">
   <inertial>
-    <origin xyz="0.003164818104754781 0.0010809996534067296 -0.002661116265664301" rpy="0 0 0"/>
-    <mass value="0.00018598053770557866"/>
-    <inertia ixx="0.0" iyy="0.0" izz="0.0" ixy="-0.0" iyz="0.0" ixz="0.0"/>
-  </inertial>
-  <visual>
-    <origin xyz="-0.060146 0.001452 -0.072623" rpy="0 0 0"/>
+    <origin xyz="0.03164392589961296 0.010807214803428875 -0.026615162656641878" rpy="0 0 0"/>
+    <mass value="0.18598053770557915"/>
+    <inertia ixx="7e-05" iyy="0.000133" izz="9.1e-05" ixy="-1.7e-05" iyz="1.5e-05" ixz="6.3e-05"/>
+  </inertial>
+  <visual>
+    <origin xyz="-0.569077 -0.066087 -0.714234" rpy="0 0 0"/>
     <geometry>
       <mesh filename="package://ros_robot_description/meshes/JawR_1.stl" scale="0.001 0.001 0.001"/>
@@ -138,5 +138,5 @@
   </visual>
   <collision>
-    <origin xyz="-0.060146 0.001452 -0.072623" rpy="0 0 0"/>
+    <origin xyz="-0.569077 -0.066087 -0.714234" rpy="0 0 0"/>
     <geometry>
       <mesh filename="package://ros_robot_description/meshes/JawR_1.stl" scale="0.001 0.001 0.001"/>
@@ -146,10 +146,10 @@
 <link name="L6_1">
   <inertial>
-    <origin xyz="0.0007874438180608817 5.134649267789226e-06 -0.0006615106867335074" rpy="0 0 0"/>
-    <mass value="0.0005095302243692644"/>
-    <inertia ixx="0.0" iyy="0.0" izz="0.0" ixy="0.0" iyz="0.0" ixz="0.0"/>
-  </inertial>
-  <visual>
-    <origin xyz="-0.059101 -0.00323 -0.073474" rpy="0 0 0"/>
+    <origin xyz="0.007879183128393752 5.456476245438435e-05 -0.006611106810297418" rpy="0 0 0"/>
+    <mass value="0.5095302243692562"/>
+    <inertia ixx="0.000845" iyy="0.000132" izz="0.000846" ixy="5e-06" iyz="0.0" ixz="3e-06"/>
+  </inertial>
+  <visual>
+    <origin xyz="-0.558618 -0.112901 -0.722736" rpy="0 0 0"/>
     <geometry>
       <mesh filename="package://ros_robot_description/meshes/L6_1.stl" scale="0.001 0.001 0.001"/>
@@ -158,5 +158,5 @@
   </visual>
   <collision>
-    <origin xyz="-0.059101 -0.00323 -0.073474" rpy="0 0 0"/>
+    <origin xyz="-0.558618 -0.112901 -0.722736" rpy="0 0 0"/>
     <geometry>
       <mesh filename="package://ros_robot_description/meshes/L6_1.stl" scale="0.001 0.001 0.001"/>
@@ -166,10 +166,10 @@
 <link name="L5_1">
   <inertial>
-    <origin xyz="0.003679575778961462 0.0017743225942793497 -0.003097887626752005" rpy="0 0 0"/>
-    <mass value="0.0014972465004237086"/>
-    <inertia ixx="0.0" iyy="0.0" izz="0.0" ixy="-0.0" iyz="0.0" ixz="0.0"/>
-  </inertial>
-  <visual>
-    <origin xyz="-0.052695 -0.001425 -0.078859" rpy="0 0 0"/>
+    <origin xyz="0.036796502641542383 0.01774244421152102 -0.03097887626757112" rpy="0 0 0"/>
+    <mass value="1.4972465004236954"/>
+    <inertia ixx="0.00089" iyy="0.001035" izz="0.00093" ixy="-7e-06" iyz="6e-06" ixz="0.000115"/>
+  </inertial>
+  <visual>
+    <origin xyz="-0.494562 -0.094855 -0.77659" rpy="0 0 0"/>
     <geometry>
       <mesh filename="package://ros_robot_description/meshes/L5_1.stl" scale="0.001 0.001 0.001"/>
@@ -178,5 +178,5 @@
   </visual>
   <collision>
-    <origin xyz="-0.052695 -0.001425 -0.078859" rpy="0 0 0"/>
+    <origin xyz="-0.494562 -0.094855 -0.77659" rpy="0 0 0"/>
     <geometry>
       <mesh filename="package://ros_robot_description/meshes/L5_1.stl" scale="0.001 0.001 0.001"/>
@@ -186,10 +186,10 @@
 <link name="L4_1">
   <inertial>
-    <origin xyz="0.007131044333540101 4.94868613514104e-05 3.801093262367772e-08" rpy="0 0 0"/>
-    <mass value="0.002311674355709378"/>
-    <inertia ixx="0.0" iyy="0.0" izz="0.0" ixy="-0.0" iyz="0.0" ixz="0.0"/>
-  </inertial>
-  <visual>
-    <origin xyz="-0.041876 -0.00315 -0.078859" rpy="0 0 0"/>
+    <origin xyz="0.07130902791151078 0.0004961184374081828 3.779030740558298e-07" rpy="0 0 0"/>
+    <mass value="2.311666481638537"/>
+    <inertia ixx="0.001409" iyy="0.00355" izz="0.003934" ixy="-1.5e-05" iyz="0.0" ixz="0.0"/>
+  </inertial>
+  <visual>
+    <origin xyz="-0.386374 -0.112103 -0.77659" rpy="0 0 0"/>
     <geometry>
       <mesh filename="package://ros_robot_description/meshes/L4_1.stl" scale="0.001 0.001 0.001"/>
@@ -198,5 +198,5 @@
   </visual>
   <collision>
-    <origin xyz="-0.041876 -0.00315 -0.078859" rpy="0 0 0"/>
+    <origin xyz="-0.386374 -0.112103 -0.77659" rpy="0 0 0"/>
     <geometry>
       <mesh filename="package://ros_robot_description/meshes/L4_1.stl" scale="0.001 0.001 0.001"/>
@@ -206,10 +206,10 @@
 <link name="L3_1">
   <inertial>
-    <origin xyz="0.0033289224763306882 0.0028030098576427936 0.0029701409399272155" rpy="0 0 0"/>
-    <mass value="0.006131958653152949"/>
-    <inertia ixx="0.0" iyy="0.0" izz="0.0" ixy="-0.0" iyz="-0.0" ixz="-0.0"/>
-  </inertial>
-  <visual>
-    <origin xyz="-0.023818 5.6e-05 -0.075259" rpy="0 0 0"/>
+    <origin xyz="0.033289969615090176 0.028027316845520345 0.029701409398982914" rpy="0 0 0"/>
+    <mass value="6.131958653186025"/>
+    <inertia ixx="0.005791" iyy="0.022845" izz="0.021796" ixy="-0.000731" iyz="-0.000651" ixz="-0.001282"/>
+  </inertial>
+  <visual>
+    <origin xyz="-0.205792 -0.080047 -0.74059" rpy="0 0 0"/>
     <geometry>
       <mesh filename="package://ros_robot_description/meshes/L3_1.stl" scale="0.001 0.001 0.001"/>
@@ -218,5 +218,5 @@
   </visual>
   <collision>
-    <origin xyz="-0.023818 5.6e-05 -0.075259" rpy="0 0 0"/>
+    <origin xyz="-0.205792 -0.080047 -0.74059" rpy="0 0 0"/>
     <geometry>
       <mesh filename="package://ros_robot_description/meshes/L3_1.stl" scale="0.001 0.001 0.001"/>
@@ -226,10 +226,10 @@
 <link name="L2_1">
   <inertial>
-    <origin xyz="-0.007949601261310342 -0.0029356112049251084 0.007574601119981435" rpy="0 0 0"/>
-    <mass value="0.0033568476748432395"/>
-    <inertia ixx="0.0" iyy="0.0" izz="0.0" ixy="-0.0" iyz="0.0" ixz="0.0"/>
-  </inertial>
-  <visual>
-    <origin xyz="-0.043616 -8.2e-05 -0.05546" rpy="0 0 0"/>
+    <origin xyz="-0.07950096268548501 -0.029355937228571147 0.07574661040954678" rpy="0 0 0"/>
+    <mass value="3.3568597539847445"/>
+    <inertia ixx="0.022491" iyy="0.044645" izz="0.022859" ixy="-4.4e-05" iyz="8.9e-05" ixz="0.021449"/>
+  </inertial>
+  <visual>
+    <origin xyz="-0.403777 -0.081424 -0.5426" rpy="0 0 0"/>
     <geometry>
       <mesh filename="package://ros_robot_description/meshes/L2_1.stl" scale="0.001 0.001 0.001"/>
@@ -238,5 +238,5 @@
   </visual>
   <collision>
-    <origin xyz="-0.043616 -8.2e-05 -0.05546" rpy="0 0 0"/>
+    <origin xyz="-0.403777 -0.081424 -0.5426" rpy="0 0 0"/>
     <geometry>
       <mesh filename="package://ros_robot_description/meshes/L2_1.stl" scale="0.001 0.001 0.001"/>
@@ -246,10 +246,10 @@
 <link name="L1_1">
   <inertial>
-    <origin xyz="0.00466115295887317 0.00035320445235190797 0.005173799268726818" rpy="0 0 0"/>
-    <mass value="0.009576700981372619"/>
-    <inertia ixx="0.0" iyy="1e-06" izz="0.0" ixy="-0.0" iyz="-0.0" ixz="-0.0"/>
-  </inertial>
-  <visual>
-    <origin xyz="-0.031833 -0.0 -0.04426" rpy="0 0 0"/>
+    <origin xyz="0.04661494578622072 0.003532294016085999 0.05173771933594512" rpy="0 0 0"/>
+    <mass value="9.576664836012535"/>
+    <inertia ixx="0.031917" iyy="0.062523" izz="0.04245" ixy="-0.00181" iyz="-0.001638" ixz="-0.023928"/>
+  </inertial>
+  <visual>
+    <origin xyz="-0.285939 -0.080604 -0.4306" rpy="0 0 0"/>
     <geometry>
       <mesh filename="package://ros_robot_description/meshes/L1_1.stl" scale="0.001 0.001 0.001"/>
@@ -258,5 +258,5 @@
   </visual>
   <collision>
-    <origin xyz="-0.031833 -0.0 -0.04426" rpy="0 0 0"/>
+    <origin xyz="-0.285939 -0.080604 -0.4306" rpy="0 0 0"/>
     <geometry>
       <mesh filename="package://ros_robot_description/meshes/L1_1.stl" scale="0.001 0.001 0.001"/>
@@ -264,12 +264,92 @@
   </collision>
 </link>
+<link name="GarbageBot_1">
+  <inertial>
+    <origin xyz="0.004156095453495663 3.839859988474803e-06 0.015000000000000034" rpy="0 0 0"/>
+    <mass value="11.613863926243594"/>
+    <inertia ixx="0.038479" iyy="0.059958" izz="0.096695" ixy="2e-06" iyz="-0.0" ixz="-0.0"/>
+  </inertial>
+  <visual>
+    <origin xyz="0.03401 -0.080602 -0.045" rpy="0 0 0"/>
+    <geometry>
+      <mesh filename="package://ros_robot_description/meshes/GarbageBot_1.stl" scale="0.001 0.001 0.001"/>
+    </geometry>
+    <material name="paint_enamel_glossy_yellow_1"/>
+  </visual>
+  <collision>
+    <origin xyz="0.03401 -0.080602 -0.045" rpy="0 0 0"/>
+    <geometry>
+      <mesh filename="package://ros_robot_description/meshes/GarbageBot_1.stl" scale="0.001 0.001 0.001"/>
+    </geometry>
+  </collision>
+</link>
+<link name="CameraFront_1">
+  <inertial>
+    <origin xyz="3.9235725490804896e-07 2.745653550351168e-07 0.03499999999999992" rpy="0 0 0"/>
+    <mass value="0.4395999999999997"/>
+    <inertia ixx="0.000238" iyy="0.000194" izz="7.3e-05" ixy="-0.0" iyz="0.0" ixz="-0.0"/>
+  </inertial>
+  <visual>
+    <origin xyz="0.30901 -0.080605 -0.91" rpy="0 0 0"/>
+    <geometry>
+      <mesh filename="package://ros_robot_description/meshes/CameraFront_1.stl" scale="0.001 0.001 0.001"/>
+    </geometry>
+    <material name="paint_enamel_glossy_red_1"/>
+  </visual>
+  <collision>
+    <origin xyz="0.30901 -0.080605 -0.91" rpy="0 0 0"/>
+    <geometry>
+      <mesh filename="package://ros_robot_description/meshes/CameraFront_1.stl" scale="0.001 0.001 0.001"/>
+    </geometry>
+  </collision>
+</link>
+<link name="CameraLeft_1">
+  <inertial>
+    <origin xyz="3.9235725468600435e-07 2.745653554098171e-07 0.03499999999999992" rpy="0 0 0"/>
+    <mass value="0.4395999999999995"/>
+    <inertia ixx="0.000194" iyy="0.000238" izz="7.3e-05" ixy="0.0" iyz="-0.0" ixz="0.0"/>
+  </inertial>
+  <visual>
+    <origin xyz="0.21901 -0.035605 -0.91" rpy="0 0 0"/>
+    <geometry>
+      <mesh filename="package://ros_robot_description/meshes/CameraLeft_1.stl" scale="0.001 0.001 0.001"/>
+    </geometry>
+    <material name="paint_enamel_glossy_red_1"/>
+  </visual>
+  <collision>
+    <origin xyz="0.21901 -0.035605 -0.91" rpy="0 0 0"/>
+    <geometry>
+      <mesh filename="package://ros_robot_description/meshes/CameraLeft_1.stl" scale="0.001 0.001 0.001"/>
+    </geometry>
+  </collision>
+</link>
+<link name="CameraRight_1">
+  <inertial>
+    <origin xyz="3.923572546582488e-07 2.745653553959393e-07 0.03499999999999992" rpy="0 0 0"/>
+    <mass value="0.4396000000000005"/>
+    <inertia ixx="0.000194" iyy="0.000238" izz="7.3e-05" ixy="0.0" iyz="-0.0" ixz="0.0"/>
+  </inertial>
+  <visual>
+    <origin xyz="0.21901 -0.125605 -0.91" rpy="0 0 0"/>
+    <geometry>
+      <mesh filename="package://ros_robot_description/meshes/CameraRight_1.stl" scale="0.001 0.001 0.001"/>
+    </geometry>
+    <material name="paint_enamel_glossy_red_1"/>
+  </visual>
+  <collision>
+    <origin xyz="0.21901 -0.125605 -0.91" rpy="0 0 0"/>
+    <geometry>
+      <mesh filename="package://ros_robot_description/meshes/CameraRight_1.stl" scale="0.001 0.001 0.001"/>
+    </geometry>
+  </collision>
+</link>
 <link name="GPS_1">
   <inertial>
-    <origin xyz="-2.3524948103079146e-07 1.056295993651712e-07 0.0015000000000000013" rpy="0 0 0"/>
-    <mass value="0.00028259999999999874"/>
-    <inertia ixx="0.0" iyy="0.0" izz="0.0" ixy="-0.0" iyz="0.0" ixz="0.0"/>
-  </inertial>
-  <visual>
-    <origin xyz="0.020662 -0.0 -0.0922" rpy="0 0 0"/>
+    <origin xyz="3.9235725490804896e-07 2.745653554930838e-07 0.015000000000000013" rpy="0 0 0"/>
+    <mass value="0.2825999999999998"/>
+    <inertia ixx="4.2e-05" iyy="5.9e-05" izz="5.9e-05" ixy="0.0" iyz="-0.0" ixz="-0.0"/>
+  </inertial>
+  <visual>
+    <origin xyz="0.25401 -0.080605 -0.91" rpy="0 0 0"/>
     <geometry>
       <mesh filename="package://ros_robot_description/meshes/GPS_1.stl" scale="0.001 0.001 0.001"/>
@@ -278,5 +358,5 @@
   </visual>
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
Commit message: .

File: urdf/ros_robot.xacro (robot description, xacro)
@@ -146,7 +146,7 @@
 <link name="L6_1">
   <inertial>
-    <origin xyz="0.007879183128393752 5.456476245438435e-05 -0.006611106810297418" rpy="0 0 0"/>
-    <mass value="0.5095302243692562"/>
-    <inertia ixx="0.000845" iyy="0.000132" izz="0.000846" ixy="5e-06" iyz="0.0" ixz="3e-06"/>
+    <origin xyz="0.008033096186199185 5.72987518178969e-05 -0.006308097141295432" rpy="0 0 0"/>
+    <mass value="0.5174654530927676"/>
+    <inertia ixx="0.000849" iyy="0.000137" izz="0.000847" ixy="5e-06" iyz="0.0" ixz="2e-06"/>
   </inertial>
   <visual>
@@ -361,4 +361,24 @@
     <geometry>
       <mesh filename="package://ros_robot_description/meshes/GPS_1.stl" scale="0.001 0.001 0.001"/>
+    </geometry>
+  </collision>
+</link>
+<link name="CameraArm_1">
+  <inertial>
+    <origin xyz="0.0032135726825279765 2.2141618967422283e-05 0.0038301783339352857" rpy="0 0 0"/>
+    <mass value="0.0039250000000000075"/>
+    <inertia ixx="0.0" iyy="0.0" izz="0.0" ixy="0.0" iyz="-0.0" ixz="-0.0"/>
+  </inertial>
+  <visual>
+    <origin xyz="-0.579297 -0.113045 -0.741936" rpy="0 0 0"/>
+    <geometry>
+      <mesh filename="package://ros_robot_description/meshes/CameraArm_1.stl" scale="0.001 0.001 0.001"/>
+    </geometry>
+    <material name="paint_enamel_glossy_red_1"/>
+  </visual>
+  <collision>
+    <origin xyz="-0.579297 -0.113045 -0.741936" rpy="0 0 0"/>
+    <geometry>
+      <mesh filename="package://ros_robot_description/meshes/CameraArm_1.stl" scale="0.001 0.001 0.001"/>
     </geometry>
   </collision>
@@ -445,15 +465,15 @@
   <child link="GarbageBot_1"/>
 </joint>
-<joint name="Rigid29" type="fixed">
+<joint name="CameraFrontMount" type="fixed">
   <origin xyz="-0.30901 0.080605 0.91" rpy="0 0 0"/>
   <parent link="base_link"/>
   <child link="CameraFront_1"/>
 </joint>
-<joint name="Rigid30" type="fixed">
+<joint name="CameraRightMount" type="fixed">
   <origin xyz="-0.21901 0.035605 0.91" rpy="0 0 0"/>
   <parent link="base_link"/>
   <child link="CameraLeft_1"/>
 </joint>
-<joint name="Rigid31" type="fixed">
+<joint name="CameraLeftMount" type="fixed">
   <origin xyz="-0.21901 0.125605 0.91" rpy="0 0 0"/>
   <parent link="base_link"/>
@@ -465,3 +485,8 @@
   <child link="GPS_1"/>
 </joint>
+<joint name="CameraArmMount" type="fixed">
+  <origin xyz="0.020679 0.000144 0.0192" rpy="0 0 0"/>
+  <parent link="L6_1"/>
+  <child link="CameraArm_1"/>
+</joint>
 </robot>
