Commit message: .

File: urdf/Sensors/ros_robot_ArmCamera.xacro (robot description, xacro)
@@ -49,8 +49,9 @@
                 </clip>
             </camera>
-            <plugin name="camera_controller" filename="libgazebo_ros_camera.so">
+            <plugin name="camera_arm_controller" filename="libgazebo_ros_camera.so">
+                <cameraName>ros_robot/camera_arm</cameraName>
                 <frame_name>CameraArm_link_optical</frame_name>
-                <imageTopicName>image_raw/camera_Arm</imageTopicName>
-                <cameraInfoTopicName>camera_info/camera_Arm</cameraInfoTopicName>
+                <imageTopicName>image_raw</imageTopicName>
+                <cameraInfoTopicName>camera_info</cameraInfoTopicName>
             </plugin>
         </sensor>

File: urdf/Sensors/ros_robot_BackCamera.xacro (robot description, xacro)
@@ -49,8 +49,9 @@
                 </clip>
             </camera>
-            <plugin name="camera_controller" filename="libgazebo_ros_camera.so">
+            <plugin name="camera_back_controller" filename="libgazebo_ros_camera.so">
+                <cameraName>ros_robot/camera_back</cameraName>
                 <frame_name>CameraBack_link_optical</frame_name>
-                <imageTopicName>image_raw/camera_Back</imageTopicName>
-                <cameraInfoTopicName>camera_info/camera_Back</cameraInfoTopicName>
+                <imageTopicName>image_raw</imageTopicName>
+                <cameraInfoTopicName>camera_info</cameraInfoTopicName>
             </plugin>
         </sensor>

File: urdf/Sensors/ros_robot_FrontCamera.xacro (robot description, xacro)
@@ -33,5 +33,5 @@
 <link name="CameraFront_link_optical"> </link>
 <gazebo reference="CameraFront_1">
-        <sensor name="camera1" type="camera">
+        <sensor name="cameraFront" type="camera">
             <pose> 0 0 0 0 0 0 </pose>
             <visualize>${visual_camera}</visualize>
@@ -49,8 +49,9 @@
                 </clip>
             </camera>
-            <plugin name="camera_controller_front" filename="libgazebo_ros_camera.so">
-                <imageTopicName>image_raw/camera_front</imageTopicName>
-                <cameraInfoTopicName>camera_info/camera_front</cameraInfoTopicName>
+            <plugin name="camera_front_controller" filename="libgazebo_ros_camera.so">
+                <cameraName>ros_robot/camera_front</cameraName>
                 <frame_name>CameraFront_link_optical</frame_name>
+                <imageTopicName>image_raw</imageTopicName>
+                <cameraInfoTopicName>camera_info</cameraInfoTopicName>
             </plugin>
         </sensor>

File: urdf/Sensors/ros_robot_LeftCamera.xacro (robot description, xacro)
@@ -49,8 +49,9 @@
                 </clip>
             </camera>
-            <plugin name="camera_controller" filename="libgazebo_ros_camera.so">
+            <plugin name="camera_left_controller" filename="libgazebo_ros_camera.so">
+                <cameraName>ros_robot/camera_left</cameraName>
                 <frame_name>CameraLeft_link_optical</frame_name>
-                <imageTopicName>image_raw/camera_left</imageTopicName>
-                <cameraInfoTopicName>camera_info/camera_left</cameraInfoTopicName>
+                <imageTopicName>image_raw</imageTopicName>
+                <cameraInfoTopicName>camera_info</cameraInfoTopicName>
             </plugin>
         </sensor>

File: urdf/Sensors/ros_robot_RightCamera.xacro (robot description, xacro)
@@ -49,8 +49,9 @@
                 </clip>
             </camera>
-            <plugin name="camera_controller" filename="libgazebo_ros_camera.so">
+            <plugin name="camera_right_controller" filename="libgazebo_ros_camera.so">
+                <cameraName>ros_robot/camera_right</cameraName>
                 <frame_name>CameraRight_link_optical</frame_name>
-                <imageTopicName>image_raw/camera_right</imageTopicName>
-                <cameraInfoTopicName>camera_info/camera_right</cameraInfoTopicName>
+                <imageTopicName>image_raw</imageTopicName>
+                <cameraInfoTopicName>camera_info</cameraInfoTopicName>
             </plugin>
         </sensor>

File: urdf/Thrusters/BackThrusterLeft.xacro (robot description, xacro)
@@ -54,4 +54,6 @@
   <child link="BackPropellerL_1"/>
   <axis xyz="1.0 0.0 0.0"/>
+  <limit effort="100" velocity="100"/>
+  <dynamics damping="0.05" friction="0.05"/>
 </joint>
 <gazebo reference="BackPropellerL_1">

File: urdf/Thrusters/BackThrusterRight.xacro (robot description, xacro)
@@ -53,4 +53,6 @@
   <child link="BackPropellerR_1"/>
   <axis xyz="1.0 0.0 0.0"/>
+  <limit effort="100" velocity="100"/>
+  <dynamics damping="0.05" friction="0.05"/>
 </joint>
 <gazebo reference="BackPropellerR_1">

File: urdf/Thrusters/CenterThruster.xacro (robot description, xacro)
@@ -14,4 +14,11 @@
     <material name="paint_enamel_glossy_red"/>
   </visual>
+<!--
+  <collision name="left_engine_vertical_axis_collision">
+      <origin rpy="0 0 0" xyz="0 0 -0.24"/>
+      <geometry>
+        <box size="0.2 0.15 0.2"/>
+      </geometry>
+    </collision>
   <collision>
     <origin xyz="0.304047 -0.080604 -0.010094" rpy="0 0 0"/>
@@ -20,4 +27,5 @@
     </geometry>
   </collision>
+-->
 </link>
 <link name="CenterPropeller_1">
@@ -34,4 +42,12 @@
     <material name="abs_white"/>
   </visual>
+<!--
+  <collision name="left_propeller_collision">
+    <origin rpy="0 1.57 0" xyz="0 0 0"/>
+    <geometry>
+      <cylinder length="0.18" radius="0.08"/>
+    </geometry>
+  </collision>
+  -->
   <collision>
     <origin xyz="0.264443 -0.080604 0.097906" rpy="0 0 0"/>
@@ -49,9 +65,10 @@
 </joint>
 <joint name="CenterThrusterProp" type="continuous">
-  <!--  <axis xyz="0 1.0 0"/>-->
-  <axis xyz="1.0 0.0 -0.0"/>
+  <axis xyz="1.0 0.0 0.0"/>
   <origin xyz="0.039604 0.0 -0.108" rpy="0 0 0"/>
   <parent link="CenterThruster_1"/>
   <child link="CenterPropeller_1"/>
+  <limit effort="100" velocity="100"/>
+  <dynamics damping="0.05" friction="0.05"/>
 </joint>
 <gazebo reference="CenterPropeller_1">

File: urdf/ros_robot.xacro (robot description, xacro)
@@ -10,4 +10,5 @@
 <xacro:include filename="$(find ros_robot_description)/urdf/Sensors/ros_robot_BackCamera.xacro" />
 <xacro:include filename="$(find ros_robot_description)/urdf/Sensors/ros_robot_ArmCamera.xacro" />
+<xacro:include filename="$(find ros_robot_description)/urdf/Sensors/ros_robot_rangingSensor.xacro"/>
 <xacro:include filename="$(find ros_robot_description)/urdf/Sensors/ros_robot_GpsSensor.xacro" />
 <xacro:include filename="$(find ros_robot_description)/urdf/Thrusters/CenterThruster.xacro" />
