Commit message: rework Axis

File: urdf/RobotArm/RobotArm.xacro (robot description, xacro)
@@ -3,10 +3,10 @@
 <link name="JawL_1">
   <inertial>
-    <origin xyz="0.03189007234749497 -0.010365489487497326 -0.026698581275366062" rpy="0 0 0"/>
+    <origin xyz="-0.03189029458894865 0.010364926026270288 -0.02669858127536817" rpy="0 0 0"/>
     <mass value="0.0018"/>
     <inertia ixx="7e-05" iyy="0.000135" izz="9.2e-05" ixy="1.7e-05" iyz="-1.4e-05" ixz="6.3e-05"/>
   </inertial>
   <visual>
-    <origin xyz="-0.568429 -0.159356 -0.714234" rpy="0 0 0"/>
+    <origin xyz="0.568431 0.078647 -0.714234" rpy="0 0 0"/>
     <geometry>
       <mesh filename="package://ros_robot_description/meshes/JawL_1.stl" scale="0.001 0.001 0.001"/>
@@ -15,5 +15,5 @@
   </visual>
   <collision>
-    <origin xyz="-0.568429 -0.159356 -0.714234" rpy="0 0 0"/>
+    <origin xyz="0.568431 0.078647 -0.714234" rpy="0 0 0"/>
     <geometry>
       <mesh filename="package://ros_robot_description/meshes/JawL_1.stl" scale="0.001 0.001 0.001"/>
@@ -23,10 +23,10 @@
 <link name="JawR_1">
   <inertial>
-    <origin xyz="0.03164392589961296 0.010807214803428875 -0.026615162656641878" rpy="0 0 0"/>
+    <origin xyz="-0.031644148141077966 -0.010806778264657124 -0.026615162656639213" rpy="0 0 0"/>
     <mass value="0.0018"/>
     <inertia ixx="7e-05" iyy="0.000133" izz="9.1e-05" ixy="-1.7e-05" iyz="1.5e-05" ixz="6.3e-05"/>
   </inertial>
   <visual>
-    <origin xyz="-0.569077 -0.066087 -0.714234" rpy="0 0 0"/>
+    <origin xyz="0.569079 -0.014621 -0.714234" rpy="0 0 0"/>
     <geometry>
       <mesh filename="package://ros_robot_description/meshes/JawR_1.stl" scale="0.001 0.001 0.001"/>
@@ -35,5 +35,5 @@
   </visual>
   <collision>
-    <origin xyz="-0.569077 -0.066087 -0.714234" rpy="0 0 0"/>
+    <origin xyz="0.569079 -0.014621 -0.714234" rpy="0 0 0"/>
     <geometry>
       <mesh filename="package://ros_robot_description/meshes/JawR_1.stl" scale="0.001 0.001 0.001"/>
@@ -43,10 +43,10 @@
 <link name="L6_1">
   <inertial>
-    <origin xyz="0.008033096186199185 5.72987518178969e-05 -0.006308097141295432" rpy="0 0 0"/>
+    <origin xyz="-0.00803331842765087 -5.6862213045037746e-05 -0.006308097141295432" rpy="0 0 0"/>
     <mass value="0.0018"/>
     <inertia ixx="0.000849" iyy="0.000137" izz="0.000847" ixy="5e-06" iyz="0.0" ixz="2e-06"/>
   </inertial>
   <visual>
-    <origin xyz="-0.558618 -0.112901 -0.722736" rpy="0 0 0"/>
+    <origin xyz="0.55862 0.032193 -0.722736" rpy="0 0 0"/>
     <geometry>
       <mesh filename="package://ros_robot_description/meshes/L6_1.stl" scale="0.001 0.001 0.001"/>
@@ -55,5 +55,5 @@
   </visual>
   <collision>
-    <origin xyz="-0.558618 -0.112901 -0.722736" rpy="0 0 0"/>
+    <origin xyz="0.55862 0.032193 -0.722736" rpy="0 0 0"/>
     <geometry>
       <mesh filename="package://ros_robot_description/meshes/L6_1.stl" scale="0.001 0.001 0.001"/>
@@ -63,10 +63,10 @@
 <link name="L5_1">
   <inertial>
-    <origin xyz="0.036796502641542383 0.01774244421152102 -0.03097887626757112" rpy="0 0 0"/>
+    <origin xyz="-0.036796724882995124 -0.017742007672748007 -0.0309788762675699" rpy="0 0 0"/>
     <mass value="0.0018"/>
     <inertia ixx="0.00089" iyy="0.001035" izz="0.00093" ixy="-7e-06" iyz="6e-06" ixz="0.000115"/>
   </inertial>
   <visual>
-    <origin xyz="-0.494562 -0.094855 -0.77659" rpy="0 0 0"/>
+    <origin xyz="0.494564 0.014147 -0.77659" rpy="0 0 0"/>
     <geometry>
       <mesh filename="package://ros_robot_description/meshes/L5_1.stl" scale="0.001 0.001 0.001"/>
@@ -75,5 +75,5 @@
   </visual>
   <collision>
-    <origin xyz="-0.494562 -0.094855 -0.77659" rpy="0 0 0"/>
+    <origin xyz="0.494564 0.014147 -0.77659" rpy="0 0 0"/>
     <geometry>
       <mesh filename="package://ros_robot_description/meshes/L5_1.stl" scale="0.001 0.001 0.001"/>
@@ -83,10 +83,10 @@
 <link name="L4_1">
   <inertial>
-    <origin xyz="0.07130902791151078 0.0004961184374081828 3.779030740558298e-07" rpy="0 0 0"/>
+    <origin xyz="-0.07130925015296014 -0.0004956819947762731 3.779030740558298e-07" rpy="0 0 0"/>
     <mass value="0.0018"/>
     <inertia ixx="0.001409" iyy="0.00355" izz="0.003934" ixy="-1.5e-05" iyz="0.0" ixz="0.0"/>
   </inertial>
   <visual>
-    <origin xyz="-0.386374 -0.112103 -0.77659" rpy="0 0 0"/>
+    <origin xyz="0.386376 0.031395 -0.77659" rpy="0 0 0"/>
     <geometry>
       <mesh filename="package://ros_robot_description/meshes/L4_1.stl" scale="0.001 0.001 0.001"/>
@@ -95,5 +95,5 @@
   </visual>
   <collision>
-    <origin xyz="-0.386374 -0.112103 -0.77659" rpy="0 0 0"/>
+    <origin xyz="0.386376 0.031395 -0.77659" rpy="0 0 0"/>
     <geometry>
       <mesh filename="package://ros_robot_description/meshes/L4_1.stl" scale="0.001 0.001 0.001"/>
@@ -103,10 +103,10 @@
 <link name="L3_1">
   <inertial>
-    <origin xyz="0.033289969615090176 0.028027316845520345 0.029701409398982914" rpy="0 0 0"/>
+    <origin xyz="-0.03328919185654228 -0.028027880306747386 0.029701409398983136" rpy="0 0 0"/>
     <mass value="0.0018"/>
     <inertia ixx="0.005791" iyy="0.022845" izz="0.021796" ixy="-0.000731" iyz="-0.000651" ixz="-0.001282"/>
   </inertial>
   <visual>
-    <origin xyz="-0.205792 -0.080047 -0.74059" rpy="0 0 0"/>
+    <origin xyz="0.205795 -0.000662 -0.74059" rpy="0 0 0"/>
     <geometry>
       <mesh filename="package://ros_robot_description/meshes/L3_1.stl" scale="0.001 0.001 0.001"/>
@@ -115,5 +115,5 @@
   </visual>
   <collision>
-    <origin xyz="-0.205792 -0.080047 -0.74059" rpy="0 0 0"/>
+    <origin xyz="0.205795 -0.000662 -0.74059" rpy="0 0 0"/>
     <geometry>
       <mesh filename="package://ros_robot_description/meshes/L3_1.stl" scale="0.001 0.001 0.001"/>
@@ -123,10 +123,10 @@
 <link name="L2_1">
   <inertial>
-    <origin xyz="-0.07950096268548501 -0.029355937228571147 0.07574661040954678" rpy="0 0 0"/>
+    <origin xyz="0.07950139518636501 0.029355377391545236 0.07574626013664454" rpy="0 0 0"/>
     <mass value="0.0018"/>
     <inertia ixx="0.022491" iyy="0.044645" izz="0.022859" ixy="-4.4e-05" iyz="8.9e-05" ixz="0.021449"/>
   </inertial>
   <visual>
-    <origin xyz="-0.403777 -0.081424 -0.5426" rpy="0 0 0"/>
+    <origin xyz="0.40378 0.000715 -0.5426" rpy="0 0 0"/>
     <geometry>
       <mesh filename="package://ros_robot_description/meshes/L2_1.stl" scale="0.001 0.001 0.001"/>
@@ -135,5 +135,5 @@
   </visual>
   <collision>
-    <origin xyz="-0.403777 -0.081424 -0.5426" rpy="0 0 0"/>
+    <origin xyz="0.40378 0.000715 -0.5426" rpy="0 0 0"/>
     <geometry>
       <mesh filename="package://ros_robot_description/meshes/L2_1.stl" scale="0.001 0.001 0.001"/>
@@ -143,10 +143,10 @@
 <link name="L1_1">
   <inertial>
-    <origin xyz="0.04661494578622072 0.003532294016085999 0.05173771933594512" rpy="0 0 0"/>
+    <origin xyz="-0.04661521084736314 -0.003531900009707762 0.05173767169330279" rpy="0 0 0"/>
     <mass value="0.0018"/>
     <inertia ixx="0.031917" iyy="0.062523" izz="0.04245" ixy="-0.00181" iyz="-0.001638" ixz="-0.023928"/>
   </inertial>
   <visual>
-    <origin xyz="-0.285939 -0.080604 -0.4306" rpy="0 0 0"/>
+    <origin xyz="0.285941 -0.000104 -0.4306" rpy="0 0 0"/>
     <geometry>
       <mesh filename="package://ros_robot_description/meshes/L1_1.stl" scale="0.001 0.001 0.001"/>
@@ -155,5 +155,5 @@
   </visual>
   <collision>
-    <origin xyz="-0.285939 -0.080604 -0.4306" rpy="0 0 0"/>
+    <origin xyz="0.285941 -0.000104 -0.4306" rpy="0 0 0"/>
     <geometry>
       <mesh filename="package://ros_robot_description/meshes/L1_1.stl" scale="0.001 0.001 0.001"/>
@@ -162,58 +162,58 @@
 </link>
 <joint name="JawL" type="prismatic">
-  <origin xyz="0.009811 0.046455 -0.008502" rpy="0 0 0"/>
+  <origin xyz="-0.009811 -0.046454 -0.008502" rpy="0 0 0"/>
   <parent link="L6_1"/>
   <child link="JawL_1"/>
-  <axis xyz="0.0 0.999966 0.008286"/>
+  <axis xyz="0.0 0.999966 -0.008286"/>
   <limit upper="0.005" lower="-0.003" effort="100" velocity="100"/>
 </joint>
 <joint name="JawR" type="prismatic">
-  <origin xyz="0.010459 -0.046814 -0.008502" rpy="0 0 0"/>
+  <origin xyz="-0.010459 0.046814 -0.008502" rpy="0 0 0"/>
   <parent link="L6_1"/>
   <child link="JawR_1"/>
-  <axis xyz="0.0 0.999966 0.008286"/>
+  <axis xyz="0.0 0.999966 -0.008286"/>
   <limit upper="0.0021" lower="-0.005" effort="100" velocity="100"/>
 </joint>
 <joint name="L6" type="revolute">
-  <origin xyz="0.064056 0.018046 -0.053854" rpy="0 0 0"/>
+  <origin xyz="-0.064056 -0.018046 -0.053854" rpy="0 0 0"/>
   <parent link="L5_1"/>
   <child link="L6_1"/>
-  <axis xyz="0.766026 0.005327 -0.642788"/>
+  <axis xyz="-0.766026 -0.005327 -0.642788"/>
   <limit upper="3.141593" lower="-3.141593" effort="100" velocity="100"/>
 </joint>
 <joint name="L5" type="revolute">
-  <origin xyz="0.108188 -0.017248 0.0" rpy="0 0 0"/>
+  <origin xyz="-0.108188 0.017248 0.0" rpy="0 0 0"/>
   <parent link="L4_1"/>
   <child link="L5_1"/>
-  <axis xyz="0.006953 -0.999976 -0.0"/>
+  <axis xyz="-0.006953 0.999976 -0.0"/>
   <limit upper="2.617994" lower="-1.308997" effort="100" velocity="100"/>
 </joint>
 <joint name="L4" type="revolute">
-  <origin xyz="0.180582 0.032056 0.036" rpy="0 0 0"/>
+  <origin xyz="-0.180581 -0.032057 0.036" rpy="0 0 0"/>
   <parent link="L3_1"/>
   <child link="L4_1"/>
-  <axis xyz="0.999976 0.006953 0.0"/>
+  <axis xyz="-0.999976 -0.006953 0.0"/>
   <limit upper="3.141593" lower="-3.141593" effort="100" velocity="100"/>
 </joint>
 <joint name="L3" type="revolute">
-  <origin xyz="-0.197985 -0.001377 0.19799" rpy="0 0 0"/>
+  <origin xyz="0.197985 0.001377 0.19799" rpy="0 0 0"/>
   <parent link="L2_1"/>
   <child link="L3_1"/>
-  <axis xyz="-0.006953 0.999976 0.0"/>
+  <axis xyz="0.006953 -0.999976 0.0"/>
   <limit upper="0.610865" lower="-4.101524" effort="100" velocity="100"/>
 </joint>
 <joint name="L2" type="revolute">
-  <origin xyz="0.117838 0.00082 0.112" rpy="0 0 0"/>
+  <origin xyz="-0.117839 -0.000819 0.112" rpy="0 0 0"/>
   <parent link="L1_1"/>
   <child link="L2_1"/>
-  <axis xyz="0.006953 -0.999976 -0.0"/>
+  <axis xyz="-0.006953 0.999976 -0.0"/>
   <limit upper="1.134464" lower="-3.490659" effort="100" velocity="100"/>
   <dynamics damping="100.0" friction="100.0"/>  <!--fjern denne, kun for å holde armen i ro når ingen controller -->
 </joint>
 <joint name="L1" type="revolute">
-  <origin xyz="0.285939 0.080604 0.4306" rpy="0 0 0"/>
+  <origin xyz="-0.285941 0.000104 0.4306" rpy="0 0 0"/>
   <parent link="base_link"/>
   <child link="L1_1"/>
-  <axis xyz="-0.0 -0.0 1.0"/>
+  <axis xyz="0.0 0.0 1.0"/>
   <limit upper="2.181662" lower="-2.181662" effort="100" velocity="100"/>
 </joint>

File: urdf/Sensors/ArmCamera.xacro (robot description, xacro)
@@ -3,10 +3,10 @@
 <link name="CameraArm_1">
   <inertial>
-    <origin xyz="0.0032135726825279765 2.2141618967422283e-05 0.0038301783339352857" rpy="0 0 0"/>
+    <origin xyz="-0.0032137949239799957 -2.2705080194432292e-05 0.0038301783339353968" rpy="0 0 0"/>
     <mass value="0.003"/>
     <inertia ixx="0.0" iyy="0.0" izz="0.0" ixy="0.0" iyz="-0.0" ixz="-0.0"/>
   </inertial>
   <visual>
-    <origin xyz="-0.579297 -0.113045 -0.741936" rpy="0 0 0"/>
+    <origin xyz="0.579299 0.032336 -0.741936" rpy="0 0 0"/>
     <geometry>
       <mesh filename="package://ros_robot_description/meshes/CameraArm_1.stl" scale="0.001 0.001 0.001"/>
@@ -15,5 +15,5 @@
   </visual>
   <collision>
-    <origin xyz="-0.579297 -0.113045 -0.741936" rpy="0 0 0"/>
+    <origin xyz="0.579299 0.032336 -0.741936" rpy="0 0 0"/>
     <geometry>
       <mesh filename="package://ros_robot_description/meshes/CameraArm_1.stl" scale="0.001 0.001 0.001"/>
@@ -22,5 +22,5 @@
 </link>
 <joint name="CameraArmMount" type="fixed">
-  <origin xyz="0.020679 0.000144 0.0192" rpy="0 0.523599 0"/>
+  <origin xyz="-0.020679 -0.000143 0.0192" rpy="0 0 0"/>
   <parent link="L6_1"/>
   <child link="CameraArm_1"/>

File: urdf/Sensors/BackCamera.xacro (robot description, xacro)
@@ -3,10 +3,10 @@
 <link name="CameraBack_1">
   <inertial>
-    <origin xyz="3.923572550745824e-07 2.7456535542369487e-07 0.03499999999999981" rpy="0 0 0"/>
+    <origin xyz="3.8540129290720593e-07 1.6197341744270761e-07 0.03499999999999992" rpy="0 0 0"/>
     <mass value="0.003"/>
     <inertia ixx="0.000238" iyy="0.000194" izz="7.3e-05" ixy="-0.0" iyz="0.0" ixz="0.0"/>
   </inertial>
   <visual>
-    <origin xyz="0.20901 -0.080605 -0.91" rpy="0 0 0"/>
+    <origin xyz="-0.209007 -0.000103 -0.91" rpy="0 0 0"/>
     <geometry>
       <mesh filename="package://ros_robot_description/meshes/CameraBack_1.stl" scale="0.001 0.001 0.001"/>
@@ -15,5 +15,5 @@
   </visual>
   <collision>
-    <origin xyz="0.20901 -0.080605 -0.91" rpy="0 0 0"/>
+    <origin xyz="-0.209007 -0.000103 -0.91" rpy="0 0 0"/>
     <geometry>
       <mesh filename="package://ros_robot_description/meshes/CameraBack_1.stl" scale="0.001 0.001 0.001"/>
@@ -22,5 +22,5 @@
 </link>
 <joint name="CameraBackMount" type="fixed">
-  <origin xyz="-0.20901 0.080605 0.91" rpy="0 0 0"/>
+  <origin xyz="0.209007 0.000103 0.91" rpy="0 0 0"/>
   <parent link="base_link"/>
   <child link="CameraBack_1"/>

File: urdf/Sensors/FrontCamera.xacro (robot description, xacro)
@@ -3,10 +3,10 @@
 <link name="CameraFront_1">
   <inertial>
-    <origin xyz="3.9235725490804896e-07 2.745653550351168e-07 0.03499999999999992" rpy="0 0 0"/>
+    <origin xyz="3.8540129299047265e-07 1.6197341779798711e-07 0.03500000000000025" rpy="0 0 0"/>
     <mass value="0.003"/>
     <inertia ixx="0.000238" iyy="0.000194" izz="7.3e-05" ixy="-0.0" iyz="0.0" ixz="-0.0"/>
   </inertial>
   <visual>
-    <origin xyz="0.30901 -0.080605 -0.91" rpy="0 0 0"/>
+    <origin xyz="-0.309007 -0.000103 -0.91" rpy="0 0 0"/>
     <geometry>
       <mesh filename="package://ros_robot_description/meshes/CameraFront_1.stl" scale="0.001 0.001 0.001"/>
@@ -15,5 +15,5 @@
   </visual>
   <collision>
-    <origin xyz="0.30901 -0.080605 -0.91" rpy="0 0 0"/>
+    <origin xyz="-0.309007 -0.000103 -0.91" rpy="0 0 0"/>
     <geometry>
       <mesh filename="package://ros_robot_description/meshes/CameraFront_1.stl" scale="0.001 0.001 0.001"/>
@@ -22,5 +22,5 @@
 </link>
 <joint name="CameraFrontMount" type="fixed">
-  <origin xyz="-0.30901 0.080605 0.91" rpy="0 0 3.14"/>
+  <origin xyz="0.309007 0.000103 0.91" rpy="0 0 0"/>
   <parent link="base_link"/>
   <child link="CameraFront_1"/>

File: urdf/Sensors/GpsSensor.xacro (robot description, xacro)
@@ -3,10 +3,10 @@
 <link name="GPS_1">
   <inertial>
-    <origin xyz="3.9235725490804896e-07 2.745653554930838e-07 0.015000000000000013" rpy="0 0 0"/>
+    <origin xyz="3.8540129310149496e-07 1.6197341740718644e-07 0.015000000000000013" rpy="0 0 0"/>
     <mass value="0.003"/>
     <inertia ixx="4.2e-05" iyy="5.9e-05" izz="5.9e-05" ixy="0.0" iyz="-0.0" ixz="-0.0"/>
   </inertial>
   <visual>
-    <origin xyz="0.25401 -0.080605 -0.91" rpy="0 0 0"/>
+    <origin xyz="-0.254007 -0.000103 -0.91" rpy="0 0 0"/>
     <geometry>
       <mesh filename="package://ros_robot_description/meshes/GPS_1.stl" scale="0.001 0.001 0.001"/>
@@ -15,5 +15,5 @@
   </visual>
   <collision>
-    <origin xyz="0.25401 -0.080605 -0.91" rpy="0 0 0"/>
+    <origin xyz="-0.254007 -0.000103 -0.91" rpy="0 0 0"/>
     <geometry>
       <mesh filename="package://ros_robot_description/meshes/GPS_1.stl" scale="0.001 0.001 0.001"/>
@@ -22,5 +22,5 @@
 </link>
 <joint name="gpsmount" type="fixed">
-  <origin xyz="-0.25401 0.080605 0.91" rpy="0 0 0"/>
+  <origin xyz="0.254007 0.000103 0.91" rpy="0 0 0"/>
   <parent link="base_link"/>
   <child link="GPS_1"/>

File: urdf/Sensors/LeftCamera.xacro (robot description, xacro)
@@ -3,10 +3,10 @@
 <link name="CameraLeft_1">
   <inertial>
-    <origin xyz="3.9235725468600435e-07 2.745653554098171e-07 0.03499999999999992" rpy="0 0 0"/>
+    <origin xyz="3.8540129332353956e-07 1.6197341752566263e-07 0.03500000000000014" rpy="0 0 0"/>
     <mass value="0.003"/>
     <inertia ixx="0.000194" iyy="0.000238" izz="7.3e-05" ixy="0.0" iyz="-0.0" ixz="0.0"/>
   </inertial>
   <visual>
-    <origin xyz="0.21901 -0.035605 -0.91" rpy="0 0 0"/>
+    <origin xyz="-0.219007 -0.045103 -0.91" rpy="0 0 0"/>
     <geometry>
       <mesh filename="package://ros_robot_description/meshes/CameraLeft_1.stl" scale="0.001 0.001 0.001"/>
@@ -15,5 +15,5 @@
   </visual>
   <collision>
-    <origin xyz="0.21901 -0.035605 -0.91" rpy="0 0 0"/>
+    <origin xyz="-0.219007 -0.045103 -0.91" rpy="0 0 0"/>
     <geometry>
       <mesh filename="package://ros_robot_description/meshes/CameraLeft_1.stl" scale="0.001 0.001 0.001"/>
@@ -22,5 +22,5 @@
 </link>
 <joint name="CameraLeftMount" type="fixed">
-  <origin xyz="-0.21901 0.035605 0.91" rpy="0 0 ${-pi/2}"/>
+  <origin xyz="0.219007 -0.044897 0.91" rpy="0 0 0"/>
   <parent link="base_link"/>
   <child link="CameraLeft_1"/>
@@ -32,28 +32,31 @@
 </joint>
 <link name="CameraLeft_link_optical"> </link>
+<!---->
 <gazebo reference="CameraLeft_1">
-        <sensor name="cameraLeft" type="camera">
-            <pose> 0 0 0 0 0 0 </pose>
-            <visualize>${visual_camera}</visualize>
-            <update_rate>10</update_rate>
-            <camera>
-                <horizontal_fov>1.3962634</horizontal_fov>
-                <image>
-                    <format>R8G8B8</format>
-                    <width>640</width>
-                    <height>480</height>
-                </image>
-                <clip>
-                    <near>0.05</near>
-                    <far>200</far>
-                </clip>
-            </camera>
-            <plugin name="camera_left_controller" filename="libgazebo_ros_camera.so">
-                <cameraName>ros_robot/camera_left</cameraName>
-                <frame_name>CameraLeft_link_optical</frame_name>
-                <imageTopicName>image_raw</imageTopicName>
-                <cameraInfoTopicName>camera_info</cameraInfoTopicName>
-            </plugin>
-        </sensor>
+  <plugin name="camera_left_controller" filename="libgazebo_ros_openni_kinect.so">
+    <baseline>0.2</baseline>
+    <alwaysOn>true</alwaysOn>
+    <!-- Keep this zero, update_rate in the parent <sensor> tag
+        will control the frame rate. -->
+    <updateRate>20.0</updateRate>
+    <cameraName>camera_ir</cameraName>
+    <imageTopicName>/camera/color/image_raw</imageTopicName>
+    <cameraInfoTopicName>/camera/color/camera_info</cameraInfoTopicName>
+    <depthImageTopicName>/camera/depth/image_raw</depthImageTopicName>
+    <depthImageCameraInfoTopicName>/camera/depth/camera_info</depthImageCameraInfoTopicName>
+    <pointCloudTopicName>/camera/depth/points</pointCloudTopicName>
+    <frameName>CameraLeft_link_optical</frameName>
+    <pointCloudCutoff>0.05</pointCloudCutoff>
+    <distortionK1>0</distortionK1>
+    <distortionK2>0</distortionK2>
+    <distortionK3>0</distortionK3>
+    <distortionT1>0</distortionT1>
+    <distortionT2>0</distortionT2>
+    <CxPrime>0</CxPrime>
+    <Cx>0</Cx>
+    <Cy>0</Cy>
+    <focalLength>0</focalLength>
+    <hackBaseline>0</hackBaseline>
+  </plugin>
 </gazebo>
 <gazebo reference="CameraLeft_1">

File: urdf/Sensors/RightCamera.xacro (robot description, xacro)
@@ -3,10 +3,10 @@
 <link name="CameraRight_1">
   <inertial>
-    <origin xyz="3.923572546582488e-07 2.745653553959393e-07 0.03499999999999992" rpy="0 0 0"/>
+    <origin xyz="3.8540129332353956e-07 1.6197341751178485e-07 0.03499999999999992" rpy="0 0 0"/>
     <mass value="0.003"/>
     <inertia ixx="0.000194" iyy="0.000238" izz="7.3e-05" ixy="0.0" iyz="-0.0" ixz="0.0"/>
   </inertial>
   <visual>
-    <origin xyz="0.21901 -0.125605 -0.91" rpy="0 0 0"/>
+    <origin xyz="-0.219007 0.044897 -0.91" rpy="0 0 0"/>
     <geometry>
       <mesh filename="package://ros_robot_description/meshes/CameraRight_1.stl" scale="0.001 0.001 0.001"/>
@@ -15,5 +15,5 @@
   </visual>
   <collision>
-    <origin xyz="0.21901 -0.125605 -0.91" rpy="0 0 0"/>
+    <origin xyz="-0.219007 0.044897 -0.91" rpy="0 0 0"/>
     <geometry>
       <mesh filename="package://ros_robot_description/meshes/CameraRight_1.stl" scale="0.001 0.001 0.001"/>
@@ -22,5 +22,5 @@
 </link>
 <joint name="CameraRightMount" type="fixed">
-  <origin xyz="-0.21901 0.125605 0.91" rpy="0 0 ${pi/2}"/>
+  <origin xyz="0.219007 0.045103 0.91" rpy="0 0 0"/>
   <parent link="base_link"/>
   <child link="CameraRight_1"/>

File: urdf/Sensors/imu_sensor.xacro (robot description, xacro)
@@ -16,14 +16,18 @@
     </inertial>
   </link>
-  <joint name="imu_joint" type="revolute">
-    <axis xyz="0 0 0"/>
-    <limit effort="1000.0" lower="0.0" upper="0" velocity="0"/>
+  <joint name="imu_joint" type="fixed">
     <origin rpy="0 0 0" xyz="0 0 0"/>
     <parent link="base_link"/>
     <child link="imu_link"/>
   </joint>
+  <joint name="magnometer_joint" type="fixed">
+    <origin xyz="0 0 0" rpy="0 0 0"/>
+    <parent link="imu_link"/>
+    <child link="magnometer_link"/>
+  </joint>
+  <link name="magnometer_link"> </link>
   <gazebo>
-    <plugin filename="libhector_gazebo_ros_imu.so" name="imu_plugin_imu_wamv">
-      <updateRate>15</updateRate>
+    <plugin filename="libhector_gazebo_ros_imu.so" name="imu_plugin">
+      <updateRate>20</updateRate>
       <bodyName>imu_link</bodyName>
       <topicName>sensors/imu/data</topicName>
@@ -46,3 +50,17 @@
     </plugin>
   </gazebo>
+  <gazebo>
+    <plugin filename="libhector_gazebo_ros_magnetic.so" name="magnetometer">
+      <updateRate>20.0</updateRate>
+      <bodyname>magnometer_link</bodyname>
+      <topicName>sensors/magnometer</topicName>
+      <referenceHeading>72.0</referenceHeading>
+      <!--<magnitude>5.7065E-5</magnitude>-->
+      <declination>12</declination>
+      <inclination>64</inclination>
+      <offset>0 0 0</offset>
+      <driftFrequency>0 0 0</driftFrequency>
+      <gaussianNoise>0 0 0</gaussianNoise>
+    </plugin>
+  </gazebo>
 </robot>
