Commit message: rework Axis

File: urdf/Thrusters/BackThrusterLeft.xacro (robot description, xacro)
@@ -3,10 +3,10 @@
 <link name="BackThrusterL_1">
   <inertial>
-    <origin xyz="0.006792471139986711 2.1826936180691092e-07 -0.15892739606734135" rpy="0 0 0"/>
+    <origin xyz="-0.00679269338143873 2.1826941126734667e-07 -0.15892739606734135" rpy="0 0 0"/>
     <mass value="1.9708306012870964"/>
     <inertia ixx="0.011921" iyy="0.012132" izz="0.000443" ixy="-0.0" iyz="-0.0" ixz="0.000811"/>
   </inertial>
   <visual>
-    <origin xyz="-0.515512 0.069396 -0.279079" rpy="0 0 0"/>
+    <origin xyz="0.515514 -0.150104 -0.279079" rpy="0 0 0"/>
     <geometry>
       <mesh filename="package://ros_robot_description/meshes/BackThrusterL_1.stl" scale="0.001 0.001 0.001"/>
@@ -15,5 +15,5 @@
   </visual>
   <collision>
-    <origin xyz="-0.515512 0.069396 -0.279079" rpy="0 0 0"/>
+    <origin xyz="0.515514 -0.150104 -0.279079" rpy="0 0 0"/>
     <geometry>
       <mesh filename="package://ros_robot_description/meshes/BackThrusterL_1.stl" scale="0.001 0.001 0.001"/>
@@ -23,10 +23,10 @@
 <link name="BackPropellerL_1">
   <inertial>
-    <origin xyz="0.02691630233499631 6.95845980332177e-06 -1.3859013972401107e-05" rpy="0 0 0"/>
+    <origin xyz="-0.02691605112418549 -6.697354491103091e-06 -1.4490021561459898e-05" rpy="0 0 0"/>
     <mass value="0.6485270682886274"/>
     <inertia ixx="0.000738" iyy="0.000497" izz="0.000497" ixy="0.0" iyz="0.0" ixz="-0.0"/>
   </inertial>
   <visual>
-    <origin xyz="-0.555117 0.069396 -0.022079" rpy="0 0 0"/>
+    <origin xyz="0.555119 -0.150104 -0.022079" rpy="0 0 0"/>
     <geometry>
       <mesh filename="package://ros_robot_description/meshes/BackPropellerL_1.stl" scale="0.001 0.001 0.001"/>
@@ -35,5 +35,5 @@
   </visual>
   <collision>
-    <origin xyz="-0.555117 0.069396 -0.022079" rpy="0 0 0"/>
+    <origin xyz="0.555119 -0.150104 -0.022079" rpy="0 0 0"/>
     <geometry>
       <mesh filename="package://ros_robot_description/meshes/BackPropellerL_1.stl" scale="0.001 0.001 0.001"/>
@@ -42,5 +42,5 @@
 </link>
 <joint name="BackThrusterL" type="revolute">
-  <origin xyz="0.515512 -0.069396 0.279079" rpy="0 0 0"/>
+  <origin xyz="-0.515514 0.150104 0.279079" rpy="0 0 0"/>
   <axis xyz="0.0 0.0 -1.0"/>
   <parent link="base_link"/>
@@ -50,8 +50,8 @@
 <!--for unknown reason, cant turn prop-->
 <joint name="BackThrusterLProp" type="continuous">
-  <origin xyz="0.039605 0.0 -0.257" rpy="0 0 0"/>
+  <origin xyz="-0.039605 0.0 -0.257" rpy="0 0 0"/>
   <parent link="BackThrusterL_1"/>
   <child link="BackPropellerL_1"/>
-  <axis xyz="1.0 0.0 0.0"/>
+  <axis xyz="-1.0 0.0 0.0"/>
   <limit effort="100" velocity="100"/>
   <dynamics damping="0.05" friction="0.05"/>

File: urdf/Thrusters/BackThrusterRight.xacro (robot description, xacro)
@@ -3,10 +3,10 @@
 <link name="BackThrusterR_1">
   <inertial>
-    <origin xyz="0.006792377549189488 -2.097044343452037e-07 -0.15892739606734108" rpy="0 0 0"/>
+    <origin xyz="-0.006792599790641174 -3.537567924427609e-07 -0.15892739606734108" rpy="0 0 0"/>
     <mass value="1.9708306012870964"/>
     <inertia ixx="0.011921" iyy="0.012132" izz="0.000443" ixy="0.0" iyz="-0.0" ixz="0.000811"/>
   </inertial>
   <visual>
-    <origin xyz="-0.513675 -0.21201 -0.279079" rpy="0 0 0"/>
+    <origin xyz="0.513677 0.131301 -0.279079" rpy="0 0 0"/>
     <geometry>
       <mesh filename="package://ros_robot_description/meshes/BackThrusterR_1.stl" scale="0.001 0.001 0.001"/>
@@ -15,5 +15,5 @@
   </visual>
   <collision>
-    <origin xyz="-0.513675 -0.21201 -0.279079" rpy="0 0 0"/>
+    <origin xyz="0.513677 0.131301 -0.279079" rpy="0 0 0"/>
     <geometry>
       <mesh filename="package://ros_robot_description/meshes/BackThrusterR_1.stl" scale="0.001 0.001 0.001"/>
@@ -23,10 +23,10 @@
 <link name="BackPropellerR_1">
   <inertial>
-    <origin xyz="0.0269162087441992 6.530486007155778e-06 -1.3859013972307432e-05" rpy="0 0 0"/>
+    <origin xyz="-0.02691595753329501 -7.269386166353087e-06 -1.4490021474883319e-05" rpy="0 0 0"/>
     <mass value="0.6485270682886274"/>
     <inertia ixx="0.000738" iyy="0.000497" izz="0.000497" ixy="0.0" iyz="0.0" ixz="-0.0"/>
   </inertial>
   <visual>
-    <origin xyz="-0.55328 -0.21201 -0.022079" rpy="0 0 0"/>
+    <origin xyz="0.553282 0.131301 -0.022079" rpy="0 0 0"/>
     <geometry>
       <mesh filename="package://ros_robot_description/meshes/BackPropellerR_1.stl" scale="0.001 0.001 0.001"/>
@@ -35,5 +35,5 @@
   </visual>
   <collision>
-    <origin xyz="-0.55328 -0.21201 -0.022079" rpy="0 0 0"/>
+    <origin xyz="0.553282 0.131301 -0.022079" rpy="0 0 0"/>
     <geometry>
       <mesh filename="package://ros_robot_description/meshes/BackPropellerR_1.stl" scale="0.001 0.001 0.001"/>
@@ -42,5 +42,5 @@
 </link>
 <joint name="BackThrusterR" type="revolute">
-  <origin xyz="0.513675 0.21201 0.279079" rpy="0 0 0"/>
+  <origin xyz="-0.513677 -0.131301 0.279079" rpy="0 0 0"/>
   <axis xyz="0.0 0.0 1.0"/>
   <parent link="base_link"/>
@@ -49,8 +49,8 @@
 </joint>
 <joint name="BackThrusterRProp" type="continuous">
-  <origin xyz="0.039605 0.0 -0.257" rpy="0 0 0"/>
+  <origin xyz="-0.039605 0.0 -0.257" rpy="0 0 0"/>
   <parent link="BackThrusterR_1"/>
   <child link="BackPropellerR_1"/>
-  <axis xyz="1.0 0.0 0.0"/>
+  <axis xyz="-1.0 0.0 0.0"/>
   <limit effort="100" velocity="100"/>
   <dynamics damping="0.05" friction="0.05"/>

File: urdf/Thrusters/CenterThruster.xacro (robot description, xacro)
@@ -3,10 +3,10 @@
 <link name="CenterThruster_1">
   <inertial>
-    <origin xyz="0.011171747345905592 2.1404408209746428e-07 -0.06436169555636481" rpy="0 0 0"/>
+    <origin xyz="-0.011171969587361441 2.2249469140611026e-07 -0.0643616955563667" rpy="0 0 0"/>
     <mass value="1.1982535523983007"/>
     <inertia ixx="0.001394" iyy="0.001546" izz="0.000303" ixy="-0.0" iyz="-0.0" ixz="8.2e-05"/>
   </inertial>
   <visual>
-    <origin xyz="0.304047 -0.080604 -0.010094" rpy="0 0 0"/>
+    <origin xyz="-0.304045 -0.000104 -0.010094" rpy="0 0 0"/>
     <geometry>
       <mesh filename="package://ros_robot_description/meshes/CenterThruster_1.stl" scale="0.001 0.001 0.001"/>
@@ -22,5 +22,5 @@
     </collision>
   <collision>
-    <origin xyz="0.304047 -0.080604 -0.010094" rpy="0 0 0"/>
+    <origin xyz="-0.304045 -0.000104 -0.010094" rpy="0 0 0"/>
     <geometry>
       <mesh filename="package://ros_robot_description/meshes/CenterThruster_1.stl" scale="0.001 0.001 0.001"/>
@@ -31,10 +31,10 @@
 <link name="CenterPropeller_1">
   <inertial>
-    <origin xyz="0.02839655475562558 6.954234524222946e-06 -1.3373438184152708e-05" rpy="0 0 0"/>
+    <origin xyz="-0.028395303528591626 -6.693132053848039e-06 -1.4004445823653788e-05" rpy="0 0 0"/>
     <mass value="0.6485270682886274"/>
     <inertia ixx="0.000738" iyy="0.000497" izz="0.000497" ixy="0.0" iyz="0.0" ixz="-0.0"/>
   </inertial>
   <visual>
-    <origin xyz="0.264443 -0.080604 0.097906" rpy="0 0 0"/>
+    <origin xyz="-0.26444 -0.000104 0.097906" rpy="0 0 0"/>
     <geometry>
       <mesh filename="package://ros_robot_description/meshes/CenterPropellerR_1.stl" scale="0.001 0.001 0.001"/>
@@ -51,5 +51,5 @@
   -->
   <collision>
-    <origin xyz="0.264443 -0.080604 0.097906" rpy="0 0 0"/>
+    <origin xyz="-0.26444 -0.000104 0.097906" rpy="0 0 0"/>
     <geometry>
       <mesh filename="package://ros_robot_description/meshes/CenterPropellerR_1.stl" scale="0.001 0.001 0.001"/>
@@ -59,5 +59,5 @@
 <joint name="CenterThruster" type="revolute">
   <axis xyz="0.0 0.0 -1.0"/>
-  <origin xyz="-0.304047 0.080604 0.010094" rpy="0 0 0"/>
+  <origin xyz="0.304045 0.000104 0.010094" rpy="0 0 0"/>
   <parent link="base_link"/>
   <child link="CenterThruster_1"/>
@@ -65,6 +65,6 @@
 </joint>
 <joint name="CenterThrusterProp" type="continuous">
-  <axis xyz="1.0 0.0 0.0"/>
-  <origin xyz="0.039604 0.0 -0.108" rpy="0 0 0"/>
+  <axis xyz="-1.0 0.0 -0.0"/>
+  <origin xyz="-0.039605 0.0 -0.108" rpy="0 0 0"/>
   <parent link="CenterThruster_1"/>
   <child link="CenterPropeller_1"/>

File: urdf/ros_robot.xacro (robot description, xacro)
@@ -20,5 +20,5 @@
 <link name="base_link">
   <inertial>
-    <origin xyz="0.044354227312182234 0.08057379028516376 0.21043007492326804" rpy="0 0 0"/>
+    <origin xyz="-0.040426671996312426 0.00016559498592984233 0.209559986591449" rpy="0 0 0"/>
     <mass value="110"/>
     <inertia ixx="0.1" iyy="0.1" izz="0.1" ixy="0" iyz="0" ixz="0"/>
@@ -40,10 +40,10 @@
 <link name="GarbageBot_1">
   <inertial>
-    <origin xyz="0.004156095453495663 3.839859988474803e-06 0.015000000000000034" rpy="0 0 0"/>
+    <origin xyz="-0.00415631769494771 -3.4033212155202414e-06 0.015000000000000027" rpy="0 0 0"/>
     <mass value="11"/>
     <inertia ixx="0.038479" iyy="0.059958" izz="0.096695" ixy="2e-06" iyz="-0.0" ixz="-0.0"/>
   </inertial>
   <visual>
-    <origin xyz="0.03401 -0.080602 -0.045" rpy="0 0 0"/>
+    <origin xyz="-0.034008 -0.000106 -0.045" rpy="0 0 0"/>
     <geometry>
       <mesh filename="package://ros_robot_description/meshes/GarbageBot_1.stl" scale="0.001 0.001 0.001"/>
@@ -52,5 +52,5 @@
   </visual>
   <collision>
-    <origin xyz="0.03401 -0.080602 -0.045" rpy="0 0 0"/>
+    <origin xyz="-0.034008 -0.000106 -0.045" rpy="0 0 0"/>
     <geometry>
       <mesh filename="package://ros_robot_description/meshes/GarbageBot_1.stl" scale="0.001 0.001 0.001"/>
@@ -60,5 +60,5 @@
 <link name="world_boat_link"/>
 <joint name="world_boat_joint" type="fixed">
-  <origin xyz="0 0 0" rpy="0 0 3.14"/>
+  <origin xyz="0 0 0" rpy="0 0 0"/>
   <parent link="world_boat_link"/>
   <child link="base_link"/>

File: worlds/testworld.xacro (robot description, xacro)
@@ -35,5 +35,5 @@
     <include>
       <name>crocodile_buoy</name>
-      <pose>10 2 0 0 0 0</pose>
+      <pose>0 1 0 0 0 0</pose>
       <uri>model://crocodile_buoy</uri>
     </include>

Commit message: RobotArmOnly added

File: urdf/RobotArm/RobotArm.xacro (robot description, xacro)
@@ -1,4 +1,24 @@
 <?xml version="1.0" ?>
 <robot name="ros_robot" xmlns:xacro="http://www.ros.org/wiki/xacro" >
+<link name="ArmBase_1">
+  <inertial>
+    <origin xyz="0.0011454041878000698 0.0011459188982486657 0.030935981147480862" rpy="0 0 0"/>
+    <mass value="23.097311942049508"/>
+    <inertia ixx="0.093308" iyy="0.093308" izz="0.170178" ixy="0.002057" iyz="-0.000107" ixz="-0.000107"/>
+  </inertial>
+  <visual>
+    <origin xyz="0.285941 -0.000104 -0.346" rpy="0 0 0"/>
+    <geometry>
+      <mesh filename="package://ros_robot_description/meshes/ArmBase_1.stl" scale="0.001 0.001 0.001"/>
+    </geometry>
+    <material name="paint_enamel_glossy_black"/>
+  </visual>
+  <collision>
+    <origin xyz="0.285941 -0.000104 -0.346" rpy="0 0 0"/>
+    <geometry>
+      <mesh filename="package://ros_robot_description/meshes/ArmBase_1.stl" scale="0.001 0.001 0.001"/>
+    </geometry>
+  </collision>
+</link>
 <link name="JawL_1">
   <inertial>
@@ -212,9 +232,14 @@
 </joint>
 <joint name="L1" type="revolute">
-  <origin xyz="-0.285941 0.000104 0.4306" rpy="0 0 0"/>
-  <parent link="base_link"/>
+  <origin xyz="0.0 0.0 0.0856" rpy="0 0 0"/>
+  <parent link="ArmBase_1"/>
   <child link="L1_1"/>
   <axis xyz="0.0 0.0 1.0"/>
   <limit upper="2.181662" lower="-2.181662" effort="100" velocity="100"/>
 </joint>
+<joint name="ArmBaseLink" type="fixed">
+  <origin xyz="-0.285941 0.000104 0.346" rpy="0 0 0"/>
+  <parent link="base_link"/>
+  <child link="ArmBase_1"/>
+</joint>
 </robot>

File: urdf/Sensors/GpsSensor.xacro (robot description, xacro)
@@ -34,5 +34,5 @@
   <gazebo>
     <plugin filename="libhector_gazebo_ros_gps.so" name="gps_plugin_gps">
-      <updateRate>15</updateRate>
+      <updateRate>1</updateRate>
       <alwaysOn>true</alwaysOn>
       <bodyName>GPS_1</bodyName>

File: urdf/Sensors/LeftCamera.xacro (robot description, xacro)
@@ -67,5 +67,5 @@
               <frameName>CameraLeft_left_link_optical</frameName>
               <pointCloudCutoff>0.4</pointCloudCutoff>
-              <pointCloudCutoffMax>3.0</pointCloudCutoffMax>-
+              <pointCloudCutoffMax>4.0</pointCloudCutoffMax>-
             </plugin>
         </sensor>

File: urdf/Sensors/RightCamera.xacro (robot description, xacro)
@@ -57,5 +57,5 @@
                   </clip>
               </camera>
-            <plugin name="kinect_plugin" filename="libgazebo_ros_openni_kinect.so">
+            <plugin name="kinect_plugin2" filename="libgazebo_ros_openni_kinect.so">
               <baseline>0.1</baseline>
               <alwaysOn>true</alwaysOn>

File: urdf/Sensors/imu_sensor.xacro (robot description, xacro)
@@ -29,5 +29,5 @@
   <gazebo>
     <plugin filename="libhector_gazebo_ros_imu.so" name="imu_plugin">
-      <updateRate>20</updateRate>
+      <updateRate>100</updateRate>
       <bodyName>imu_link</bodyName>
       <topicName>sensors/imu/data</topicName>
@@ -56,7 +56,7 @@
       <topicName>sensors/magnometer</topicName>
       <referenceHeading>72.0</referenceHeading>
-      <!--<magnitude>5.7065E-5</magnitude>-->
-      <declination>12</declination>
-      <inclination>64</inclination>
+      <magnitude>5.7065E-5</magnitude>
+      <declination>12.3</declination>
+      <inclination>64.2</inclination>
       <offset>0 0 0</offset>
       <driftFrequency>0 0 0</driftFrequency>

File: urdf/ros_robot.xacro (robot description, xacro)
@@ -18,7 +18,8 @@
 <xacro:include filename="$(find ros_robot_description)/urdf/RobotArm/RobotArm.xacro" />
 <xacro:include filename="$(find ros_robot_description)/urdf/RobotArm/RobotArm.gazebo" />
+<xacro:include filename="$(find ros_robot_description)/urdf/RobotArm/RobotArm.trans" />
 <link name="base_link">
   <inertial>
-    <origin xyz="-0.040426671996312426 0.00016559498592984233 0.209559986591449" rpy="0 0 0"/>
+    <origin xyz="-0.03405684570032273 0.00013676637886197947 0.20520744004115304" rpy="0 0 0"/>
     <mass value="110"/>
     <inertia ixx="0.1" iyy="0.1" izz="0.1" ixy="0" iyz="0" ixz="0"/>

Commit message: Added plugin and transmissions for robotarm

File: urdf/RobotArm/RobotArm.xacro (robot description, xacro)
@@ -243,3 +243,84 @@
   <child link="ArmBase_1"/>
 </joint>
+<!--Transmission-->
+<transmission name="JawL_Tran">
+    <type>transmission_interface/SimpleTransmission</type>
+    <joint name="JawL">
+      <hardwareInterface>hardware_interface/PositionJointInterface</hardwareInterface>
+    </joint>
+    <actuator name="JawL_Motor">
+      <hardwareInterface>hardware_interface/PositionJointInterface</hardwareInterface>
+      <mechanicalReduction>1</mechanicalReduction>
+    </actuator>
+  </transmission>
+<transmission name="JawR_Tran">
+    <type>transmission_interface/SimpleTransmission</type>
+    <joint name="JawR">
+      <hardwareInterface>hardware_interface/PositionJointInterface</hardwareInterface>
+    </joint>
+    <actuator name="JawR_Motor">
+      <hardwareInterface>hardware_interface/PositionJointInterface</hardwareInterface>
+      <mechanicalReduction>1</mechanicalReduction>
+    </actuator>
+  </transmission>
+<transmission name="L6_Tran">
+    <type>transmission_interface/SimpleTransmission</type>
+    <joint name="L6">
+      <hardwareInterface>hardware_interface/PositionJointInterface</hardwareInterface>
+    </joint>
+    <actuator name="L6_Motor">
+      <hardwareInterface>hardware_interface/PositionJointInterface</hardwareInterface>
+      <mechanicalReduction>1</mechanicalReduction>
+    </actuator>
+  </transmission>
+<transmission name="L5_Tran">
+    <type>transmission_interface/SimpleTransmission</type>
+    <joint name="L5">
+      <hardwareInterface>hardware_interface/PositionJointInterface</hardwareInterface>
+    </joint>
+    <actuator name="L5_Motor">
+      <hardwareInterface>hardware_interface/PositionJointInterface</hardwareInterface>
+      <mechanicalReduction>1</mechanicalReduction>
+    </actuator>
+  </transmission>
+<transmission name="L4_Tran">
+    <type>transmission_interface/SimpleTransmission</type>
+    <joint name="L4">
+      <hardwareInterface>hardware_interface/PositionJointInterface</hardwareInterface>
+    </joint>
+    <actuator name="L4_Motor">
+      <hardwareInterface>hardware_interface/PositionJointInterface</hardwareInterface>
+      <mechanicalReduction>1</mechanicalReduction>
+    </actuator>
+  </transmission>
+<transmission name="L3_Tran">
+    <type>transmission_interface/SimpleTransmission</type>
+    <joint name="L3">
+      <hardwareInterface>hardware_interface/PositionJointInterface</hardwareInterface>
+    </joint>
+    <actuator name="L3_Motor">
+      <hardwareInterface>hardware_interface/PositionJointInterface</hardwareInterface>
+      <mechanicalReduction>1</mechanicalReduction>
+    </actuator>
+  </transmission>
+<transmission name="L2_Tran">
+    <type>transmission_interface/SimpleTransmission</type>
+    <joint name="L2">
+      <hardwareInterface>hardware_interface/PositionJointInterface</hardwareInterface>
+    </joint>
+    <actuator name="L2_Motor">
+      <hardwareInterface>hardware_interface/PositionJointInterface</hardwareInterface>
+      <mechanicalReduction>1</mechanicalReduction>
+    </actuator>
+  </transmission>
+ <transmission name="L1_Tran">
+    <type>transmission_interface/SimpleTransmission</type>
+    <joint name="L1">
+      <hardwareInterface>hardware_interface/PositionJointInterface</hardwareInterface>
+    </joint>
+    <actuator name="L1_Motor">
+      <hardwareInterface>hardware_interface/PositionJointInterface</hardwareInterface>
+      <mechanicalReduction>1</mechanicalReduction>
+    </actuator>
+  </transmission>
 </robot>

Commit message: Removed transmissions from xacro file

File: urdf/RobotArm/RobotArm.xacro (robot description, xacro)
@@ -243,84 +243,3 @@
   <child link="ArmBase_1"/>
 </joint>
-<!--Transmission-->
-<transmission name="JawL_Tran">
-    <type>transmission_interface/SimpleTransmission</type>
-    <joint name="JawL">
-      <hardwareInterface>hardware_interface/PositionJointInterface</hardwareInterface>
-    </joint>
-    <actuator name="JawL_Motor">
-      <hardwareInterface>hardware_interface/PositionJointInterface</hardwareInterface>
-      <mechanicalReduction>1</mechanicalReduction>
-    </actuator>
-  </transmission>
-<transmission name="JawR_Tran">
-    <type>transmission_interface/SimpleTransmission</type>
-    <joint name="JawR">
-      <hardwareInterface>hardware_interface/PositionJointInterface</hardwareInterface>
-    </joint>
-    <actuator name="JawR_Motor">
-      <hardwareInterface>hardware_interface/PositionJointInterface</hardwareInterface>
-      <mechanicalReduction>1</mechanicalReduction>
-    </actuator>
-  </transmission>
-<transmission name="L6_Tran">
-    <type>transmission_interface/SimpleTransmission</type>
-    <joint name="L6">
-      <hardwareInterface>hardware_interface/PositionJointInterface</hardwareInterface>
-    </joint>
-    <actuator name="L6_Motor">
-      <hardwareInterface>hardware_interface/PositionJointInterface</hardwareInterface>
-      <mechanicalReduction>1</mechanicalReduction>
-    </actuator>
-  </transmission>
-<transmission name="L5_Tran">
-    <type>transmission_interface/SimpleTransmission</type>
-    <joint name="L5">
-      <hardwareInterface>hardware_interface/PositionJointInterface</hardwareInterface>
-    </joint>
-    <actuator name="L5_Motor">
-      <hardwareInterface>hardware_interface/PositionJointInterface</hardwareInterface>
-      <mechanicalReduction>1</mechanicalReduction>
-    </actuator>
-  </transmission>
-<transmission name="L4_Tran">
-    <type>transmission_interface/SimpleTransmission</type>
-    <joint name="L4">
-      <hardwareInterface>hardware_interface/PositionJointInterface</hardwareInterface>
-    </joint>
-    <actuator name="L4_Motor">
-      <hardwareInterface>hardware_interface/PositionJointInterface</hardwareInterface>
-      <mechanicalReduction>1</mechanicalReduction>
-    </actuator>
-  </transmission>
-<transmission name="L3_Tran">
-    <type>transmission_interface/SimpleTransmission</type>
-    <joint name="L3">
-      <hardwareInterface>hardware_interface/PositionJointInterface</hardwareInterface>
-    </joint>
-    <actuator name="L3_Motor">
-      <hardwareInterface>hardware_interface/PositionJointInterface</hardwareInterface>
-      <mechanicalReduction>1</mechanicalReduction>
-    </actuator>
-  </transmission>
-<transmission name="L2_Tran">
-    <type>transmission_interface/SimpleTransmission</type>
-    <joint name="L2">
-      <hardwareInterface>hardware_interface/PositionJointInterface</hardwareInterface>
-    </joint>
-    <actuator name="L2_Motor">
-      <hardwareInterface>hardware_interface/PositionJointInterface</hardwareInterface>
-      <mechanicalReduction>1</mechanicalReduction>
-    </actuator>
-  </transmission>
- <transmission name="L1_Tran">
-    <type>transmission_interface/SimpleTransmission</type>
-    <joint name="L1">
-      <hardwareInterface>hardware_interface/PositionJointInterface</hardwareInterface>
-    </joint>
-    <actuator name="L1_Motor">
-      <hardwareInterface>hardware_interface/PositionJointInterface</hardwareInterface>
-      <mechanicalReduction>1</mechanicalReduction>
-    </actuator>
-  </transmission>
 </robot>

Commit message: Updated PID parameters

File: urdf/RobotArm/RobotArm.xacro (robot description, xacro)
@@ -229,5 +229,4 @@
   <axis xyz="-0.006953 0.999976 -0.0"/>
   <limit upper="1.134464" lower="-3.490659" effort="100" velocity="100"/>
-  <dynamics damping="100.0" friction="100.0"/>  <!--fjern denne, kun for å holde armen i ro når ingen controller -->
 </joint>
 <joint name="L1" type="revolute">
